File: PCB/PCB KiCad/power.kicad_sch (KiCad schematic)
At the start: 5 parts, among them U3 AMS1117-3.3

Commit message: pre route
Parts:
- removed C13: 10u, Capacitor_SMD:C_0805_2012Metric_Pad1.18x1.45mm_HandSolder, symbol Device:C
- removed U3: AMS1117-3.3, Package_TO_SOT_SMD:SOT-223-3_TabPin2, symbol Regulator_Linear:AMS1117-3.3
- renumbered C14 to C12, C15 to C13
Other:
- note removed: "Main Power Supply +5V"
Changed lines of the file:
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@@
     (company "Plastic Scanner")
-  )
-  (junction (at 173.99 63.5) (diameter 0) (color 0 0 0 0)
   )
   (junction (at 219.71 63.5) (diameter 0) (color 0 0 0 0)
@@
   (junction (at 227.33 63.5) (diameter 0) (color 0 0 0 0)
   )
-  (junction (at 108.585 76.2) (diameter 0) (color 0 0 0 0)
-  )
-  (junction (at 200.66 63.5) (diameter 0) (color 0 0 0 0)
-  )
   (junction (at 223.52 78.74) (diameter 0) (color 0 0 0 0)
   )
   (wire (pts (xy 219.71 74.93) (xy 219.71 78.74))
-    (stroke (width 0) (type default))
-  )
-  (wire (pts (xy 173.99 71.12) (xy 173.99 78.74))
-    (stroke (width 0) (type default))
-  )
-  (wire (pts (xy 83.82 49.53) (xy 83.82 76.2))
-    (stroke (width 0) (type default))
-  )
-  (wire (pts (xy 173.99 53.34) (xy 173.99 63.5))
     (stroke (width 0) (type default))
   )
@@
     (stroke (width 0) (type default))
   )
-  (wire (pts (xy 173.99 63.5) (xy 181.61 63.5))
-    (stroke (width 0) (type default))
-  )
   (wire (pts (xy 227.33 78.74) (xy 223.52 78.74))
     (stroke (width 0) (type default))
   )
-  (wire (pts (xy 196.85 63.5) (xy 200.66 63.5))
-    (stroke (width 0) (type default))
-  )
   (wire (pts (xy 227.33 74.93) (xy 227.33 78.74))
-    (stroke (width 0) (type default))
-  )
-  (wire (pts (xy 189.23 71.12) (xy 189.23 78.74))
     (stroke (width 0) (type default))
   )
@@
     (stroke (width 0) (type default))
   )
-  (wire (pts (xy 83.82 76.2) (xy 108.585 76.2))
-    (stroke (width 0) (type default))
-  )
-  (text "Main Power Supply +5V" (at 35.56 38.1 0)
-    (effects (font (size 3 3)) (justify left bottom))
-  )
   (text "+3.3v" (at 195.58 39.37 0)
     (effects (font (size 3 3)) (justify left bottom))
@@
     )
   )
-  (global_label "5v_RAW" (shape input) (at 173.99 53.34 90) (fields_autoplaced)
-    (effects (font (size 1.27 1.27)) (justify left))
-    (property "Intersheetrefs" "${INTERSHEET_REFS}" (at 173.99 43.4795 90)
-      (effects (font (size 1.27 1.27)) (justify left) hide)
-    )
-  )
-  (global_label "5v_RAW" (shape input) (at 83.82 49.53 90) (fields_autoplaced)
-    (effects (font (size 1.27 1.27)) (justify left))
-    (property "Intersheetrefs" "${INTERSHEET_REFS}" (at 83.82 39.6695 90)
-      (effects (font (size 1.27 1.27)) (justify left) hide)
-    )
-  )
   (symbol (lib_id "Device:C") (at 227.33 71.12 0) (unit 1)
     (in_bom yes) (on_board yes) (dnp no) (fields_autoplaced)
-    (property "Reference" "C15" (at 231.14 69.8499 0)
+    (property "Reference" "C13" (at 231.14 69.8499 0)
       (effects (font (size 1.27 1.27)) (justify left))
     )
@@
       (project "PCB KiCad"
         (path "/a818e058-3544-4da8-96fb-1a428660711f/5869e7b3-0d61-455b-97ad-e4e8b4829f27"
-          (reference "C15") (unit 1)
-        )
-      )
-    )
-  )
-  (symbol (lib_id "power:PWR_FLAG") (at 108.585 76.2 0) (mirror x) (unit 1)
-    (in_bom yes) (on_board yes) (dnp no) (fields_autoplaced)
-    (property "Reference" "#FLG01" (at 108.585 78.105 0)
-      (effects (font (size 1.27 1.27)) hide)
-    )
-    (property "Value" "PWR_FLAG" (at 108.585 81.28 0)
-      (effects (font (size 1.27 1.27)))
-    )
-    (property "Footprint" "" (at 108.585 76.2 0)
-      (effects (font (size 1.27 1.27)) hide)
-    )
-    (property "Datasheet" "~" (at 108.585 76.2 0)
-      (effects (font (size 1.27 1.27)) hide)
-    )
-    (pin "1")
-    (instances
-      (project "PCB KiCad"
-        (path "/a818e058-3544-4da8-96fb-1a428660711f/5869e7b3-0d61-455b-97ad-e4e8b4829f27"
-          (reference "#FLG01") (unit 1)
+          (reference "C13") (unit 1)
         )
       )
@@
   (symbol (lib_id "power:GND") (at 223.52 78.74 0) (unit 1)
     (in_bom yes) (on_board yes) (dnp no) (fields_autoplaced)
-    (property "Reference" "#PWR025" (at 223.52 85.09 0)
+    (property "Reference" "#PWR012" (at 223.52 85.09 0)
       (effects (font (size 1.27 1.27)) hide)
     )
@@
       (project "PCB KiCad"
         (path "/a818e058-3544-4da8-96fb-1a428660711f/5869e7b3-0d61-455b-97ad-e4e8b4829f27"
-          (reference "#PWR025") (unit 1)
+          (reference "#PWR012") (unit 1)
         )
       )
@@
   (symbol (lib_id "Device:C") (at 219.71 71.12 0) (mirror x) (unit 1)
     (in_bom yes) (on_board yes) (dnp no) (fields_autoplaced)
-    (property "Reference" "C14" (at 215.9 69.8499 0)
+    (property "Reference" "C12" (at 215.9 69.8499 0)
       (effects (font (size 1.27 1.27)) (justify right))
     )
@@
       (project "PCB KiCad"
         (path "/a818e058-3544-4da8-96fb-1a428660711f/5869e7b3-0d61-455b-97ad-e4e8b4829f27"
-          (reference "C14") (unit 1)
-        )
-      )
-    )
-  )
-  (symbol (lib_id "Device:C") (at 173.99 67.31 0) (unit 1)
-    (in_bom yes) (on_board yes) (dnp no) (fields_autoplaced)
-    (property "Reference" "C13" (at 177.8 66.0399 0)
-      (effects (font (size 1.27 1.27)) (justify left))
-    )
-    (property "Value" "10u" (at 177.8 68.5799 0)
-      (effects (font (size 1.27 1.27)) (justify left))
-    )
-    (property "Footprint" "Capacitor_SMD:C_0805_2012Metric_Pad1.18x1.45mm_HandSolder" (at 174.9552 71.12 0)
-      (effects (font (size 1.27 1.27)) hide)
-    )
-    (property "Datasheet" "~" (at 173.99 67.31 0)
-      (effects (font (size 1.27 1.27)) hide)
-    )
-    (pin "1")
-    (pin "2")
-    (instances
-      (project "PCB KiCad"
-        (path "/a818e058-3544-4da8-96fb-1a428660711f/5869e7b3-0d61-455b-97ad-e4e8b4829f27"
-          (reference "C13") (unit 1)
-        )
-      )
-    )
-  )
-  (symbol (lib_id "power:+5V") (at 108.585 76.2 0) (unit 1)
-    (in_bom yes) (on_board yes) (dnp no) (fields_autoplaced)
-    (property "Reference" "#PWR022" (at 108.585 80.01 0)
-      (effects (font (size 1.27 1.27)) hide)
-    )
-    (property "Value" "+5V" (at 108.585 71.12 0)
-      (effects (font (size 1.27 1.27)))
-    )
-    (property "Footprint" "" (at 108.585 76.2 0)
-      (effects (font (size 1.27 1.27)) hide)
-    )
-    (property "Datasheet" "" (at 108.585 76.2 0)
-      (effects (font (size 1.27 1.27)) hide)
-    )
-    (pin "1")
-    (instances
-      (project "PCB KiCad"
-        (path "/a818e058-3544-4da8-96fb-1a428660711f/5869e7b3-0d61-455b-97ad-e4e8b4829f27"
-          (reference "#PWR022") (unit 1)
+          (reference "C12") (unit 1)
         )
       )
@@
   (symbol (lib_id "power:+3.3V") (at 239.395 56.515 0) (unit 1)
     (in_bom yes) (on_board yes) (dnp no) (fields_autoplaced)
-    (property "Reference" "#PWR026" (at 239.395 60.325 0)
+    (property "Reference" "#PWR013" (at 239.395 60.325 0)
       (effects (font (size 1.27 1.27)) hide)
     )
@@
       (project "PCB KiCad"
         (path "/a818e058-3544-4da8-96fb-1a428660711f/5869e7b3-0d61-455b-97ad-e4e8b4829f27"
-          (reference "#PWR026") (unit 1)
+          (reference "#PWR013") (unit 1)
         )
       )
-    )
-  )
-  (symbol (lib_id "Regulator_Linear:AMS1117-3.3") (at 189.23 63.5 0) (unit 1)
-    (in_bom yes) (on_board yes) (dnp no) (fields_autoplaced)
-    (property "Reference" "U3" (at 189.23 55.88 0)
-      (effects (font (size 1.27 1.27)))
-    )
-    (property "Value" "AMS1117-3.3" (at 189.23 58.42 0)
-      (effects (font (size 1.27 1.27)))
-    )
-    (property "Footprint" "Package_TO_SOT_SMD:SOT-223-3_TabPin2" (at 189.23 58.42 0)
-      (effects (font (size 1.27 1.27)) hide)
-    )
-    (property "Datasheet" "http://www.advanced-monolithic.com/pdf/ds1117.pdf" (at 191.77 69.85 0)
-      (effects (font (size 1.27 1.27)) hide)
-    )
-    (pin "1")
-    (pin "2")
-    (pin "3")
-    (instances
-      (project "PCB KiCad"
-        (path "/a818e058-3544-4da8-96fb-1a428660711f/5869e7b3-0d61-455b-97ad-e4e8b4829f27"
-          (reference "U3") (unit 1)
-        )
-      )
-    )
-  )
-  (symbol (lib_id "power:GND") (at 189.23 78.74 0) (unit 1)
-    (in_bom yes) (on_board yes) (dnp no) (fields_autoplaced)
-    (property "Reference" "#PWR024" (at 189.23 85.09 0)
-      (effects (font (size 1.27 1.27)) hide)
-    )
-    (property "Value" "GND" (at 189.23 83.82 0)
-      (effects (font (size 1.27 1.27)))
-    )
-    (property "Footprint" "" (at 189.23 78.74 0)
-      (effects (font (size 1.27 1.27)) hide)
-    )
-    (property "Datasheet" "" (at 189.23 78.74 0)
-      (effects (font (size 1.27 1.27)) hide)
-    )
-    (pin "1")
-    (instances
-      (project "PCB KiCad"
-        (path "/a818e058-3544-4da8-96fb-1a428660711f/5869e7b3-0d61-455b-97ad-e4e8b4829f27"
-          (reference "#PWR024") (unit 1)
-        )
-      )
-    )
-  )
-  (symbol (lib_id "power:GND") (at 173.99 78.74 0) (unit 1)
-    (in_bom yes) (on_board yes) (dnp no) (fields_autoplaced)
-    (property "Reference" "#PWR023" (at 173.99 85.09 0)
-      (effects (font (size 1.27 1.27)) hide)
-    )
-    (property "Value" "GND" (at 173.99 83.82 0)
-      (effects (font (size 1.27 1.27)))
-    )
-    (property "Footprint" "" (at 173.99 78.74 0)
-      (effects (font (size 1.27 1.27)) hide)
-    )
-    (property "Datasheet" "" (at 173.99 78.74 0)
-      (effects (font (size 1.27 1.27)) hide)
-    )
-    (pin "1")
-    (instances
-      (project "PCB KiCad"
-        (path "/a818e058-3544-4da8-96fb-1a428660711f/5869e7b3-0d61-455b-97ad-e4e8b4829f27"
-          (reference "#PWR023") (unit 1)
-        )
-      )
