File: PCB/PCB KiCad/led.kicad_sch (KiCad schematic)
At the start: 21 parts, among them J4 Conn_01x04, J5 Conn_01x04, U4 TLC59208FIPWR

Commit message: pre route
Parts:
- removed R14: 1k, Resistor_SMD:R_0805_2012Metric_Pad1.20x1.40mm_HandSolder, symbol Device:R
- renumbered C16 to C14, D11 to D10, D4 to D3, D5 to D4, D6 to D5, D7 to D6, D8 to D7, D9 to D8, D10 to D9, J4 to J3, J5 to J4, R17 to R10, R18 to R11, R19 to R12, R20 to R13, R21 to R14, R22 to R15, R15 to R8, R16 to R9, U4 to U3
Connections:
- net LED_RESET: no longer names the net of U3.13 (~{RESET})
- no-connect marks 0 -> 1
