File: PCB/PCB KiCad/sensor.kicad_sch (KiCad schematic)
At the start: 12 parts, among them U1 OPA2376AID

Commit message: routed!
Parts:
- D1: footprint Diode_SMD:D_1206_3216Metric_Pad1.42x1.75mm_HandSolder -> Diode_THT:D_A-405_P2.54mm_Vertical_KathodeUp
Changed lines of the file:
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@@
+    (stroke (width 0) (type default))
+  )
+  (wire (pts (xy 34.29 100.33) (xy 33.02 100.33))
     (stroke (width 0) (type default))
   )
@@
     (stroke (width 0) (type default))
   )
+  (wire (pts (xy 34.29 102.87) (xy 34.29 100.33))
+    (stroke (width 0) (type default))
+  )
   (wire (pts (xy 110.49 132.08) (xy 140.97 132.08))
     (stroke (width 0) (type default))
@@
     (stroke (width 0) (type default))
   )
-  (wire (pts (xy 34.29 100.33) (xy 34.29 102.87))
-    (stroke (width 0) (type default))
-  )
   (wire (pts (xy 76.835 123.19) (xy 102.87 123.19))
     (stroke (width 0) (type default))
@@
   )
   (wire (pts (xy 76.835 63.5) (xy 105.41 63.5))
-    (stroke (width 0) (type default))
-  )
-  (wire (pts (xy 33.02 100.33) (xy 34.29 100.33))
     (stroke (width 0) (type default))
   )
@@
       (effects (font (size 1.27 1.27)) (justify right))
     )
-    (property "Footprint" "Diode_SMD:D_1206_3216Metric_Pad1.42x1.75mm_HandSolder" (at 33.02 96.52 0)
-      (effects (font (size 1.27 1.27)) hide)
-    )
+    (property "Footprint" "Diode_THT:D_A-405_P2.54mm_Vertical_KathodeUp" (at 33.02 96.52 0)
+      (effects (font (size 1.27 1.27)) hide)
+    )
